Commit message: modify joints properties

File: serving_arm/manipulator_description/urdf/manipulator_description.urdf (robot description, URDF)
Before this commit: robot manipulator_description, 8 links, 7 joints
Joints:
- joint link1_joint: limit (none) -> lower=-2.61799 upper=0.349066 effort=1.5 velocity=5; type continuous -> revolute
- joint link2_joint: limit (none) -> lower=-0.349066 upper=2.61799 effort=1.5 velocity=5; type continuous -> revolute
- joint link3_joint: limit (none) -> lower=-0.349066 upper=2.61799 effort=1.5 velocity=5; type continuous -> revolute
- joint rotate_joint: limit (none) -> lower=-4.71239 upper=4.71239 effort=1.5 velocity=5; type continuous -> revolute

Commit message: modify gripper_joint

File: serving_arm/manipulator_description/urdf/manipulator_description.urdf (robot description, URDF)
Before this commit: robot manipulator_description, 8 links, 7 joints
Joints:
- joint gripper_joint: origin xyz=0.155 0 0 rpy=0 0 0 -> xyz=0.13 0 0 rpy=0 0 0
